File: fab/meenie-panel.kicad_pcb (KiCad board)
At the start: 8 copper layers, 89.8 x 92 mm, 2107 parts, among them J1_01 USB-C 16P sink, J1_02 USB-C 16P sink, J1_03 USB-C 16P sink, J1_04 USB-C 16P sink, J1_05 USB-C 16P sink, J1_06 USB-C 16P sink, J1_07 USB-C 16P sink, J1_08 USB-C 16P sink, J1_09 USB-C 16P sink, J1_10 USB-C 16P sink, J1_11 USB-C 16P sink, J1_12 USB-C 16P sink, J1_13 USB-C 16P sink, J1_14 USB-C 16P sink, J1_15 USB-C 16P sink, J1_16 USB-C 16P sink, J1_17 USB-C 16P sink, J1_18 USB-C 16P sink, J1_19 USB-C 16P sink, J1_20 USB-C 16P sink, J1_21 USB-C 16P sink, J1_22 USB-C 16P sink, J1_23 USB-C 16P sink, J1_24 USB-C 16P sink, J1_25 USB-C 16P sink, J1_26 USB-C 16P sink, J1_27 USB-C 16P sink, J1_28 USB-C 16P sink, J1_29 USB-C 16P sink, J1_30 USB-C 16P sink, J1_31 USB-C 16P sink, J1_32 USB-C 16P sink, J1_33 USB-C 16P sink, J1_34 USB-C 16P sink, J1_35 USB-C 16P sink, SW1_01 GSNANOT000102, SW1_02 GSNANOT000102, SW1_03 GSNANOT000102, SW1_04 GSNANOT000102, SW1_05 GSNANOT000102, SW1_06 GSNANOT000102, SW1_07 GSNANOT000102, SW1_08 GSNANOT000102, SW1_09 GSNANOT000102, SW1_10 GSNANOT000102, SW1_11 GSNANOT000102, SW1_12 GSNANOT000102, SW1_13 GSNANOT000102, SW1_14 GSNANOT000102, SW1_15 GSNANOT000102, SW1_16 GSNANOT000102, SW1_17 GSNANOT000102, SW1_18 GSNANOT000102, SW1_19 GSNANOT000102, SW1_20 GSNANOT000102, SW1_21 GSNANOT000102, SW1_22 GSNANOT000102, SW1_23 GSNANOT000102, SW1_24 GSNANOT000102, SW1_25 GSNANOT000102, SW1_26 GSNANOT000102, SW1_27 GSNANOT000102, SW1_28 GSNANOT000102, SW1_29 GSNANOT000102, SW1_30 GSNANOT000102, SW1_31 GSNANOT000102, SW1_32 GSNANOT000102, SW1_33 GSNANOT000102, SW1_34 GSNANOT000102, SW1_35 GSNANOT000102, U1_01 nRF52840-QIAA-R, U1_02 nRF52840-QIAA-R, U1_03 nRF52840-QIAA-R, U1_04 nRF52840-QIAA-R, U1_05 nRF52840-QIAA-R, U1_06 nRF52840-QIAA-R, U1_07 nRF52840-QIAA-R, U1_08 nRF52840-QIAA-R, U1_09 nRF52840-QIAA-R, U1_10 nRF52840-QIAA-R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

Commit message: Fab Ready
Parts:
- C21_01, C21_02, C21_03, C21_04, C21_05, C21_06, C21_07, C21_08, C21_09, C21_10, C21_11, C21_12, C21_13, C21_14, C21_15, C21_16, C21_17, C21_18, C21_19, C21_20, C21_21, C21_22, C21_23, C21_24, C21_25, C21_26, C21_27, C21_28, C21_29, C21_30, C21_31, C21_32, C21_33, C21_34, C21_35: value 820pF -> 820pF C0G 5%
- C6_01, C6_02, C6_03, C6_04, C6_05, C6_06, C6_07, C6_08, C6_09, C6_10, C6_11, C6_12, C6_13, C6_14, C6_15, C6_16, C6_17, C6_18, C6_19, C6_20, C6_21, C6_22, C6_23, C6_24, C6_25, C6_26, C6_27, C6_28, C6_29, C6_30, C6_31, C6_32, C6_33, C6_34, C6_35: value 10uF -> 4.7uF; footprint meenie:C0402 -> meenie:C0603
- C8_01, C8_02, C8_03, C8_04, C8_05, C8_06, C8_07, C8_08, C8_09, C8_10, C8_11, C8_12, C8_13, C8_14, C8_15, C8_16, C8_17, C8_18, C8_19, C8_20, C8_21, C8_22, C8_23, C8_24, C8_25, C8_26, C8_27, C8_28, C8_29, C8_30, C8_31, C8_32, C8_33, C8_34, C8_35: value 1.0uF -> 100nF
- D1_01, D1_02, D1_03, D1_04, D1_05, D1_06, D1_07, D1_08, D1_09, D1_10, D1_11, D1_12, D1_13, D1_14, D1_15, D1_16, D1_17, D1_18, D1_19, D1_20, D1_21, D1_22, D1_23, D1_24, D1_25, D1_26, D1_27, D1_28, D1_29, D1_30, D1_31, D1_32, D1_33, D1_34, D1_35, D4_01, D4_02, D4_03, D4_04, D4_05, D4_06, D4_07, D4_08, D4_09, D4_10, D4_11, D4_12, D4_13, D4_14, D4_15, D4_16, D4_17, D4_18, D4_19, D4_20, D4_21, D4_22, D4_23, D4_24, D4_25, D4_26, D4_27, D4_28, D4_29, D4_30, D4_31, D4_32, D4_33, D4_34, D4_35: moved to F.Cu
- D2_01, D2_02, D2_03, D2_04, D2_05, D2_06, D2_07, D2_08, D2_09, D2_10, D2_11, D2_12, D2_13, D2_14, D2_15, D2_16, D2_17, D2_18, D2_19, D2_20, D2_21, D2_22, D2_23, D2_24, D2_25, D2_26, D2_27, D2_28, D2_29, D2_30, D2_31, D2_32, D2_33, D2_34, D2_35: value TPD1E6B06DPLR -> ESD441DPLR
- MB1, MB10, MB100, MB101, MB102, MB103, MB104, MB105, MB106, MB107, MB108, MB109, MB11, MB110, MB111, MB112, MB113, MB114, MB115, MB116, MB117, MB118, MB119, MB12, MB120, MB121, MB122, MB123, MB124, MB125, MB126, MB127, MB128, MB129, MB13, MB130, MB131, MB132, MB133, MB134, MB135, MB136, MB137, MB138, MB139, MB14, MB140, MB141, MB142, MB143, MB144, MB145, MB146, MB147, MB148, MB149, MB15, MB150, MB151, MB152, MB153, MB154, MB155, MB156, MB157, MB158, MB159, MB16, MB160, MB161, MB162, MB163, MB164, MB165, MB166, MB167, MB168, MB169, MB17, MB170, MB171, MB172, MB173, MB174, MB175, MB176, MB177, MB178, MB179, MB18, MB180, MB181, MB182, MB183, MB184, MB185, MB186, MB187, MB188, MB189, MB19, MB190, MB191, MB192, MB193, MB194, MB195, MB196, MB197, MB198, MB199, MB2, MB20, MB200, MB201, MB202, MB203, MB204, MB205, MB206, MB207, MB208, MB209, MB21, MB210, MB211, MB212, MB213, MB214, MB215, MB216, MB217, MB218, MB219, MB22, MB220, MB221, MB222, MB223, MB224, MB225, MB226, MB227, MB228, MB229, MB23, MB230, MB231, MB232, MB233, MB234, MB235, MB236, MB237, MB238, MB239, MB24, MB240, MB241, MB242, MB243, MB244, MB245, MB246, MB247, MB248, MB249, MB25, MB250, MB251, MB252, MB253, MB254, MB255, MB256, MB257, MB258, MB259, MB26, MB260, MB261, MB262, MB263, MB264, MB265, MB266, MB267, MB268, MB269, MB27, MB270, MB271, MB272, MB273, MB274, MB275, MB276, MB277, MB278, MB279, MB28, MB280, MB281, MB282, MB283, MB284, MB285, MB286, MB287, MB288, MB289, MB29, MB290, MB291, MB292, MB293, MB294, MB295, MB296, MB297, MB298, MB299, MB3, MB30, MB300, MB301, MB302, MB303, MB304, MB305, MB306, MB307, MB308, MB309, MB31, MB310, MB311, MB312, MB313, MB314, MB315, MB316, MB317, MB318, MB319, MB32, MB320, MB321, MB322, MB323, MB324, MB325, MB326, MB327, MB328, MB329, MB33, MB330, MB331, MB332, MB333, MB334, MB335, MB336, MB337, MB338, MB339, MB34, MB340, MB341, MB342, MB343, MB344, MB345, MB346, MB347, MB348, MB349, MB35, MB350, MB36, MB37, MB38, MB39, MB4, MB40, MB41, MB42, MB43, MB44, MB45, MB46, MB47, MB48, MB49, MB5, MB50, MB51, MB52, MB53, MB54, MB55, MB56, MB57, MB58, MB59, MB6, MB60, MB61, MB62, MB63, MB64, MB65, MB66, MB67, MB68, MB69, MB7, MB70, MB71, MB72, MB73, MB74, MB75, MB76, MB77, MB78, MB79, MB8, MB80, MB81, MB82, MB83, MB84, MB85, MB86, MB87, MB88, MB89, MB9, MB90, MB91, MB92, MB93, MB94, MB95, MB96, MB97, MB98, MB99: value NPTH 0.6mm -> NPTH 0.5mm; footprint panel:NPTH_0.6 -> panel:NPTH_0.5
- moved D4_01 7.46 mm to (114.5, 185.4), turned to 270 degrees
- moved D4_02 7.46 mm to (130.1, 185.4), turned to 270 degrees
- moved D4_03 7.46 mm to (145.7, 185.4), turned to 270 degrees
- moved D4_04 7.46 mm to (161.3, 185.4), turned to 270 degrees
- moved D4_06 7.46 mm to (114.5, 174.0), turned to 270 degrees
- moved D4_07 7.46 mm to (130.1, 174.0), turned to 270 degrees
- moved D4_08 7.46 mm to (145.7, 174.0), turned to 270 degrees
- moved D4_09 7.46 mm to (161.3, 174.0), turned to 270 degrees
- moved D4_21 7.46 mm to (114.5, 139.7), turned to 270 degrees
- moved D4_22 7.46 mm to (130.1, 139.7), turned to 270 degrees
- moved D4_23 7.46 mm to (145.7, 139.7), turned to 270 degrees
- moved D4_24 7.46 mm to (161.3, 139.7), turned to 270 degrees
- moved D4_26 7.46 mm to (114.5, 128.3), turned to 270 degrees
- moved D4_27 7.46 mm to (130.1, 128.3), turned to 270 degrees
- moved D4_28 7.46 mm to (145.7, 128.3), turned to 270 degrees
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Connections:
- net P0.05 renamed P1.05
- net P0.11 renamed P1.06
- net P0.13 renamed P1.01
- net P0.27 renamed P1.07
- net P0.31 renamed P0.02
- E6_01 pad 1: P1.04 -> P1.03
- E6_02 pad 1: P1.04 -> P1.03
- E6_03 pad 1: P1.04 -> P1.03
- E6_04 pad 1: P1.04 -> P1.03
- E6_05 pad 1: P1.04 -> P1.03
- E6_06 pad 1: P1.04 -> P1.03
- E6_07 pad 1: P1.04 -> P1.03
- E6_08 pad 1: P1.04 -> P1.03
- E6_09 pad 1: P1.04 -> P1.03
- E6_10 pad 1: P1.04 -> P1.03
- E6_11 pad 1: P1.04 -> P1.03
- E6_12 pad 1: P1.04 -> P1.03
- E6_13 pad 1: P1.04 -> P1.03
- E6_14 pad 1: P1.04 -> P1.03
- E6_15 pad 1: P1.04 -> P1.03
- E6_16 pad 1: P1.04 -> P1.03
- E6_17 pad 1: P1.04 -> P1.03
- E6_18 pad 1: P1.04 -> P1.03
- E6_19 pad 1: P1.04 -> P1.03
- E6_20 pad 1: P1.04 -> P1.03
- E6_21 pad 1: P1.04 -> P1.03
- E6_22 pad 1: P1.04 -> P1.03
- E6_23 pad 1: P1.04 -> P1.03
- E6_24 pad 1: P1.04 -> P1.03
- E6_25 pad 1: P1.04 -> P1.03
- E6_26 pad 1: P1.04 -> P1.03
- E6_27 pad 1: P1.04 -> P1.03
- E6_28 pad 1: P1.04 -> P1.03
- E6_29 pad 1: P1.04 -> P1.03
- E6_30 pad 1: P1.04 -> P1.03
- E6_31 pad 1: P1.04 -> P1.03
- E6_32 pad 1: P1.04 -> P1.03
- E6_33 pad 1: P1.04 -> P1.03
- E6_34 pad 1: P1.04 -> P1.03
- E6_35 pad 1: P1.04 -> P1.03
- E8_01 pad 1: P1.10 -> P1.15
- E8_02 pad 1: P1.10 -> P1.15
- E8_03 pad 1: P1.10 -> P1.15
- E8_04 pad 1: P1.10 -> P1.15
- E8_05 pad 1: P1.10 -> P1.15
- E8_06 pad 1: P1.10 -> P1.15
- E8_07 pad 1: P1.10 -> P1.15
- E8_08 pad 1: P1.10 -> P1.15
- E8_09 pad 1: P1.10 -> P1.15
- E8_10 pad 1: P1.10 -> P1.15
- E8_11 pad 1: P1.10 -> P1.15
- E8_12 pad 1: P1.10 -> P1.15
- E8_13 pad 1: P1.10 -> P1.15
- E8_14 pad 1: P1.10 -> P1.15
- E8_15 pad 1: P1.10 -> P1.15
- E8_16 pad 1: P1.10 -> P1.15
- E8_17 pad 1: P1.10 -> P1.15
- E8_18 pad 1: P1.10 -> P1.15
- E8_19 pad 1: P1.10 -> P1.15
- E8_20 pad 1: P1.10 -> P1.15
- E8_21 pad 1: P1.10 -> P1.15
- E8_22 pad 1: P1.10 -> P1.15
- E8_23 pad 1: P1.10 -> P1.15
- E8_24 pad 1: P1.10 -> P1.15
- E8_25 pad 1: P1.10 -> P1.15
- E8_26 pad 1: P1.10 -> P1.15
- E8_27 pad 1: P1.10 -> P1.15
- E8_28 pad 1: P1.10 -> P1.15
- E8_29 pad 1: P1.10 -> P1.15
- E8_30 pad 1: P1.10 -> P1.15
- E8_31 pad 1: P1.10 -> P1.15
- E8_32 pad 1: P1.10 -> P1.15
- E8_33 pad 1: P1.10 -> P1.15
- E8_34 pad 1: P1.10 -> P1.15
- E8_35 pad 1: P1.10 -> P1.15
- E9_01 pad 1: P1.11 -> P1.12
- E9_02 pad 1: P1.11 -> P1.12
- E9_03 pad 1: P1.11 -> P1.12
- E9_04 pad 1: P1.11 -> P1.12
- E9_05 pad 1: P1.11 -> P1.12
- E9_06 pad 1: P1.11 -> P1.12
- E9_07 pad 1: P1.11 -> P1.12
- E9_08 pad 1: P1.11 -> P1.12
- E9_09 pad 1: P1.11 -> P1.12
- E9_10 pad 1: P1.11 -> P1.12
- E9_11 pad 1: P1.11 -> P1.12
- E9_12 pad 1: P1.11 -> P1.12
- E9_13 pad 1: P1.11 -> P1.12
- E9_14 pad 1: P1.11 -> P1.12
- E9_15 pad 1: P1.11 -> P1.12
- E9_16 pad 1: P1.11 -> P1.12
- E9_17 pad 1: P1.11 -> P1.12
- E9_18 pad 1: P1.11 -> P1.12
- E9_19 pad 1: P1.11 -> P1.12
- E9_20 pad 1: P1.11 -> P1.12
- E9_21 pad 1: P1.11 -> P1.12
- E9_22 pad 1: P1.11 -> P1.12
- E9_23 pad 1: P1.11 -> P1.12
- E9_24 pad 1: P1.11 -> P1.12
- E9_25 pad 1: P1.11 -> P1.12
- E9_26 pad 1: P1.11 -> P1.12
- E9_27 pad 1: P1.11 -> P1.12
- E9_28 pad 1: P1.11 -> P1.12
- E9_29 pad 1: P1.11 -> P1.12
- E9_30 pad 1: P1.11 -> P1.12
- E9_31 pad 1: P1.11 -> P1.12
- E9_32 pad 1: P1.11 -> P1.12
- E9_33 pad 1: P1.11 -> P1.12
- E9_34 pad 1: P1.11 -> P1.12
- E9_35 pad 1: P1.11 -> P1.12
- U1_01 pad A14: P1.10 -> P1.15
- U1_01 pad A16: P1.15 -> P1.13
- U1_01 pad A20: P0.03 -> P1.10
- U1_01 pad B13: P0.28 -> P0.03
- U1_01 pad B17: P1.11 -> P1.12
- U1_01 pad B19: P1.12 -> P1.11
- U1_01 pad U24: P0.12 -> P1.04
- U1_01 pad V23: P1.04 -> P1.03
- U1_02 pad A14: P1.10 -> P1.15
- U1_02 pad A16: P1.15 -> P1.13
- U1_02 pad A20: P0.03 -> P1.10
- U1_02 pad B13: P0.28 -> P0.03
- U1_02 pad B17: P1.11 -> P1.12
- U1_02 pad B19: P1.12 -> P1.11
- U1_02 pad U24: P0.12 -> P1.04
- U1_02 pad V23: P1.04 -> P1.03
- U1_03 pad A14: P1.10 -> P1.15
- U1_03 pad A16: P1.15 -> P1.13
- U1_03 pad A20: P0.03 -> P1.10
- U1_03 pad B13: P0.28 -> P0.03
- U1_03 pad B17: P1.11 -> P1.12
- U1_03 pad B19: P1.12 -> P1.11
- U1_03 pad U24: P0.12 -> P1.04
- U1_03 pad V23: P1.04 -> P1.03
- U1_04 pad A14: P1.10 -> P1.15
- U1_04 pad A16: P1.15 -> P1.13
- U1_04 pad A20: P0.03 -> P1.10
- U1_04 pad B13: P0.28 -> P0.03
- U1_04 pad B17: P1.11 -> P1.12
- U1_04 pad B19: P1.12 -> P1.11
- U1_04 pad U24: P0.12 -> P1.04
- U1_04 pad V23: P1.04 -> P1.03
- U1_05 pad A14: P1.10 -> P1.15
- U1_05 pad A16: P1.15 -> P1.13
- U1_05 pad A20: P0.03 -> P1.10
- U1_05 pad B13: P0.28 -> P0.03
- U1_05 pad B17: P1.11 -> P1.12
- U1_05 pad B19: P1.12 -> P1.11
- U1_05 pad U24: P0.12 -> P1.04
- U1_05 pad V23: P1.04 -> P1.03
- U1_06 pad A14: P1.10 -> P1.15
- U1_06 pad A16: P1.15 -> P1.13
- U1_06 pad A20: P0.03 -> P1.10
- U1_06 pad B13: P0.28 -> P0.03
- U1_06 pad B17: P1.11 -> P1.12
- U1_06 pad B19: P1.12 -> P1.11
- U1_06 pad U24: P0.12 -> P1.04
- U1_06 pad V23: P1.04 -> P1.03
- U1_07 pad A14: P1.10 -> P1.15
- U1_07 pad A16: P1.15 -> P1.13
- U1_07 pad A20: P0.03 -> P1.10
- U1_07 pad B13: P0.28 -> P0.03
- U1_07 pad B17: P1.11 -> P1.12
- U1_07 pad B19: P1.12 -> P1.11
- U1_07 pad U24: P0.12 -> P1.04
- U1_07 pad V23: P1.04 -> P1.03
- U1_08 pad A14: P1.10 -> P1.15
- U1_08 pad A16: P1.15 -> P1.13
- U1_08 pad A20: P0.03 -> P1.10
- U1_08 pad B13: P0.28 -> P0.03
- U1_08 pad B17: P1.11 -> P1.12
- U1_08 pad B19: P1.12 -> P1.11
- U1_08 pad U24: P0.12 -> P1.04
- U1_08 pad V23: P1.04 -> P1.03
- U1_09 pad A14: P1.10 -> P1.15
- U1_09 pad A16: P1.15 -> P1.13
- U1_09 pad A20: P0.03 -> P1.10
- U1_09 pad B13: P0.28 -> P0.03
- U1_09 pad B17: P1.11 -> P1.12
- U1_09 pad B19: P1.12 -> P1.11
- U1_09 pad U24: P0.12 -> P1.04
- U1_09 pad V23: P1.04 -> P1.03
- U1_10 pad A14: P1.10 -> P1.15
- U1_10 pad A16: P1.15 -> P1.13
- U1_10 pad A20: P0.03 -> P1.10
- U1_10 pad B13: P0.28 -> P0.03
- U1_10 pad B17: P1.11 -> P1.12
- U1_10 pad B19: P1.12 -> P1.11
- U1_10 pad U24: P0.12 -> P1.04
- U1_10 pad V23: P1.04 -> P1.03
- U1_11 pad A14: P1.10 -> P1.15
- U1_11 pad A16: P1.15 -> P1.13
- U1_11 pad A20: P0.03 -> P1.10
- U1_11 pad B13: P0.28 -> P0.03
- U1_11 pad B17: P1.11 -> P1.12
- U1_11 pad B19: P1.12 -> P1.11
- U1_11 pad U24: P0.12 -> P1.04
- U1_11 pad V23: P1.04 -> P1.03
- U1_12 pad A14: P1.10 -> P1.15
- U1_12 pad A16: P1.15 -> P1.13
- U1_12 pad A20: P0.03 -> P1.10
- U1_12 pad B13: P0.28 -> P0.03
- U1_12 pad B17: P1.11 -> P1.12
- U1_12 pad B19: P1.12 -> P1.11
- U1_12 pad U24: P0.12 -> P1.04
- U1_12 pad V23: P1.04 -> P1.03
- U1_13 pad A14: P1.10 -> P1.15
- U1_13 pad A16: P1.15 -> P1.13
- U1_13 pad A20: P0.03 -> P1.10
- U1_13 pad B13: P0.28 -> P0.03
- U1_13 pad B17: P1.11 -> P1.12
- U1_13 pad B19: P1.12 -> P1.11
- U1_13 pad U24: P0.12 -> P1.04
- U1_13 pad V23: P1.04 -> P1.03
- U1_14 pad A14: P1.10 -> P1.15
- U1_14 pad A16: P1.15 -> P1.13
- U1_14 pad A20: P0.03 -> P1.10
- U1_14 pad B13: P0.28 -> P0.03
- U1_14 pad B17: P1.11 -> P1.12
- U1_14 pad B19: P1.12 -> P1.11
- U1_14 pad U24: P0.12 -> P1.04
- U1_14 pad V23: P1.04 -> P1.03
- U1_15 pad A14: P1.10 -> P1.15
- U1_15 pad A16: P1.15 -> P1.13
- U1_15 pad A20: P0.03 -> P1.10
- U1_15 pad B13: P0.28 -> P0.03
- U1_15 pad B17: P1.11 -> P1.12
- U1_15 pad B19: P1.12 -> P1.11
- U1_15 pad U24: P0.12 -> P1.04
- U1_15 pad V23: P1.04 -> P1.03
- U1_16 pad A14: P1.10 -> P1.15
- U1_16 pad A16: P1.15 -> P1.13
- U1_16 pad A20: P0.03 -> P1.10
- U1_16 pad B13: P0.28 -> P0.03
- U1_16 pad B17: P1.11 -> P1.12
- U1_16 pad B19: P1.12 -> P1.11
- U1_16 pad U24: P0.12 -> P1.04
- U1_16 pad V23: P1.04 -> P1.03
- U1_17 pad A14: P1.10 -> P1.15
- U1_17 pad A16: P1.15 -> P1.13
- U1_17 pad A20: P0.03 -> P1.10
- U1_17 pad B13: P0.28 -> P0.03
- U1_17 pad B17: P1.11 -> P1.12
- U1_17 pad B19: P1.12 -> P1.11
- U1_17 pad U24: P0.12 -> P1.04
- U1_17 pad V23: P1.04 -> P1.03
- U1_18 pad A14: P1.10 -> P1.15
- U1_18 pad A16: P1.15 -> P1.13
- U1_18 pad A20: P0.03 -> P1.10
- U1_18 pad B13: P0.28 -> P0.03
- U1_18 pad B17: P1.11 -> P1.12
- U1_18 pad B19: P1.12 -> P1.11
- U1_18 pad U24: P0.12 -> P1.04
- U1_18 pad V23: P1.04 -> P1.03
- U1_19 pad A14: P1.10 -> P1.15
- U1_19 pad A16: P1.15 -> P1.13
- U1_19 pad A20: P0.03 -> P1.10
- U1_19 pad B13: P0.28 -> P0.03
- U1_19 pad B17: P1.11 -> P1.12
- U1_19 pad B19: P1.12 -> P1.11
- U1_19 pad U24: P0.12 -> P1.04
- U1_19 pad V23: P1.04 -> P1.03
- U1_20 pad A14: P1.10 -> P1.15
- U1_20 pad A16: P1.15 -> P1.13
- U1_20 pad A20: P0.03 -> P1.10
- U1_20 pad B13: P0.28 -> P0.03
- U1_20 pad B17: P1.11 -> P1.12
- U1_20 pad B19: P1.12 -> P1.11
- U1_20 pad U24: P0.12 -> P1.04
- U1_20 pad V23: P1.04 -> P1.03
- U1_21 pad A14: P1.10 -> P1.15
- U1_21 pad A16: P1.15 -> P1.13
- U1_21 pad A20: P0.03 -> P1.10
- U1_21 pad B13: P0.28 -> P0.03
- U1_21 pad B17: P1.11 -> P1.12
- U1_21 pad B19: P1.12 -> P1.11
- U1_21 pad U24: P0.12 -> P1.04
- U1_21 pad V23: P1.04 -> P1.03
- U1_22 pad A14: P1.10 -> P1.15
- U1_22 pad A16: P1.15 -> P1.13
- U1_22 pad A20: P0.03 -> P1.10
- U1_22 pad B13: P0.28 -> P0.03
- U1_22 pad B17: P1.11 -> P1.12
- U1_22 pad B19: P1.12 -> P1.11
- U1_22 pad U24: P0.12 -> P1.04
- U1_22 pad V23: P1.04 -> P1.03
- U1_23 pad A14: P1.10 -> P1.15
- U1_23 pad A16: P1.15 -> P1.13
- U1_23 pad A20: P0.03 -> P1.10
- U1_23 pad B13: P0.28 -> P0.03
- U1_23 pad B17: P1.11 -> P1.12
- U1_23 pad B19: P1.12 -> P1.11
- U1_23 pad U24: P0.12 -> P1.04
- U1_23 pad V23: P1.04 -> P1.03
- U1_24 pad A14: P1.10 -> P1.15
- U1_24 pad A16: P1.15 -> P1.13
- U1_24 pad A20: P0.03 -> P1.10
- U1_24 pad B13: P0.28 -> P0.03
- U1_24 pad B17: P1.11 -> P1.12
- U1_24 pad B19: P1.12 -> P1.11
- U1_24 pad U24: P0.12 -> P1.04
- U1_24 pad V23: P1.04 -> P1.03
- U1_25 pad A14: P1.10 -> P1.15
- U1_25 pad A16: P1.15 -> P1.13
- U1_25 pad A20: P0.03 -> P1.10
- U1_25 pad B13: P0.28 -> P0.03
- U1_25 pad B17: P1.11 -> P1.12
- U1_25 pad B19: P1.12 -> P1.11
- U1_25 pad U24: P0.12 -> P1.04
- U1_25 pad V23: P1.04 -> P1.03
- U1_26 pad A14: P1.10 -> P1.15
- U1_26 pad A16: P1.15 -> P1.13
- U1_26 pad A20: P0.03 -> P1.10
- U1_26 pad B13: P0.28 -> P0.03
- U1_26 pad B17: P1.11 -> P1.12
- U1_26 pad B19: P1.12 -> P1.11
- U1_26 pad U24: P0.12 -> P1.04
- U1_26 pad V23: P1.04 -> P1.03
- U1_27 pad A14: P1.10 -> P1.15
- U1_27 pad A16: P1.15 -> P1.13
- U1_27 pad A20: P0.03 -> P1.10
- U1_27 pad B13: P0.28 -> P0.03
- U1_27 pad B17: P1.11 -> P1.12
- U1_27 pad B19: P1.12 -> P1.11
- U1_27 pad U24: P0.12 -> P1.04
- U1_27 pad V23: P1.04 -> P1.03
- U1_28 pad A14: P1.10 -> P1.15
- U1_28 pad A16: P1.15 -> P1.13
- U1_28 pad A20: P0.03 -> P1.10
- U1_28 pad B13: P0.28 -> P0.03
- U1_28 pad B17: P1.11 -> P1.12
- U1_28 pad B19: P1.12 -> P1.11
- U1_28 pad U24: P0.12 -> P1.04
- U1_28 pad V23: P1.04 -> P1.03
- U1_29 pad A14: P1.10 -> P1.15
- U1_29 pad A16: P1.15 -> P1.13
- U1_29 pad A20: P0.03 -> P1.10
- U1_29 pad B13: P0.28 -> P0.03
- U1_29 pad B17: P1.11 -> P1.12
- U1_29 pad B19: P1.12 -> P1.11
- U1_29 pad U24: P0.12 -> P1.04
- U1_29 pad V23: P1.04 -> P1.03
- U1_30 pad A14: P1.10 -> P1.15
- U1_30 pad A16: P1.15 -> P1.13
- U1_30 pad A20: P0.03 -> P1.10
- U1_30 pad B13: P0.28 -> P0.03
- U1_30 pad B17: P1.11 -> P1.12
- U1_30 pad B19: P1.12 -> P1.11
- U1_30 pad U24: P0.12 -> P1.04
- U1_30 pad V23: P1.04 -> P1.03
- U1_31 pad A14: P1.10 -> P1.15
- U1_31 pad A16: P1.15 -> P1.13
- U1_31 pad A20: P0.03 -> P1.10
- U1_31 pad B13: P0.28 -> P0.03
- U1_31 pad B17: P1.11 -> P1.12
- U1_31 pad B19: P1.12 -> P1.11
- U1_31 pad U24: P0.12 -> P1.04
- U1_31 pad V23: P1.04 -> P1.03
- U1_32 pad A14: P1.10 -> P1.15
- U1_32 pad A16: P1.15 -> P1.13
- U1_32 pad A20: P0.03 -> P1.10
- U1_32 pad B13: P0.28 -> P0.03
- U1_32 pad B17: P1.11 -> P1.12
- U1_32 pad B19: P1.12 -> P1.11
- U1_32 pad U24: P0.12 -> P1.04
- U1_32 pad V23: P1.04 -> P1.03
- U1_33 pad A14: P1.10 -> P1.15
- U1_33 pad A16: P1.15 -> P1.13
- U1_33 pad A20: P0.03 -> P1.10
- U1_33 pad B13: P0.28 -> P0.03
- U1_33 pad B17: P1.11 -> P1.12
- U1_33 pad B19: P1.12 -> P1.11
- U1_33 pad U24: P0.12 -> P1.04
- U1_33 pad V23: P1.04 -> P1.03
- U1_34 pad A14: P1.10 -> P1.15
- U1_34 pad A16: P1.15 -> P1.13
- U1_34 pad A20: P0.03 -> P1.10
- U1_34 pad B13: P0.28 -> P0.03
- U1_34 pad B17: P1.11 -> P1.12
- U1_34 pad B19: P1.12 -> P1.11
- U1_34 pad U24: P0.12 -> P1.04
- U1_34 pad V23: P1.04 -> P1.03
- U1_35 pad A14: P1.10 -> P1.15
- U1_35 pad A16: P1.15 -> P1.13
- U1_35 pad A20: P0.03 -> P1.10
- U1_35 pad B13: P0.28 -> P0.03
- U1_35 pad B17: P1.11 -> P1.12
- U1_35 pad B19: P1.12 -> P1.11
- U1_35 pad U24: P0.12 -> P1.04
- U1_35 pad V23: P1.04 -> P1.03
- W2_01 pad 1: P1.12 -> P1.11
- W2_02 pad 1: P1.12 -> P1.11
- W2_03 pad 1: P1.12 -> P1.11
- W2_04 pad 1: P1.12 -> P1.11
- W2_05 pad 1: P1.12 -> P1.11
- W2_06 pad 1: P1.12 -> P1.11
- W2_07 pad 1: P1.12 -> P1.11
- W2_08 pad 1: P1.12 -> P1.11
- W2_09 pad 1: P1.12 -> P1.11
- W2_10 pad 1: P1.12 -> P1.11
- W2_11 pad 1: P1.12 -> P1.11
- W2_12 pad 1: P1.12 -> P1.11
- W2_13 pad 1: P1.12 -> P1.11
- W2_14 pad 1: P1.12 -> P1.11
- W2_15 pad 1: P1.12 -> P1.11
- W2_16 pad 1: P1.12 -> P1.11
- W2_17 pad 1: P1.12 -> P1.11
- W2_18 pad 1: P1.12 -> P1.11
- W2_19 pad 1: P1.12 -> P1.11
- W2_20 pad 1: P1.12 -> P1.11
- W2_21 pad 1: P1.12 -> P1.11
- W2_22 pad 1: P1.12 -> P1.11
- W2_23 pad 1: P1.12 -> P1.11
- W2_24 pad 1: P1.12 -> P1.11
- W2_25 pad 1: P1.12 -> P1.11
- W2_26 pad 1: P1.12 -> P1.11
- W2_27 pad 1: P1.12 -> P1.11
- W2_28 pad 1: P1.12 -> P1.11
- W2_29 pad 1: P1.12 -> P1.11
- W2_30 pad 1: P1.12 -> P1.11
- W2_31 pad 1: P1.12 -> P1.11
- W2_32 pad 1: P1.12 -> P1.11
- W2_33 pad 1: P1.12 -> P1.11
- W2_34 pad 1: P1.12 -> P1.11
- W2_35 pad 1: P1.12 -> P1.11
- W4_01 pad 1: P1.15 -> P1.13
- W4_02 pad 1: P1.15 -> P1.13
- W4_03 pad 1: P1.15 -> P1.13
- W4_04 pad 1: P1.15 -> P1.13
- W4_05 pad 1: P1.15 -> P1.13
- W4_06 pad 1: P1.15 -> P1.13
- W4_07 pad 1: P1.15 -> P1.13
- W4_08 pad 1: P1.15 -> P1.13
- W4_09 pad 1: P1.15 -> P1.13
- W4_10 pad 1: P1.15 -> P1.13
- W4_11 pad 1: P1.15 -> P1.13
- W4_12 pad 1: P1.15 -> P1.13
- W4_13 pad 1: P1.15 -> P1.13
- W4_14 pad 1: P1.15 -> P1.13
- W4_15 pad 1: P1.15 -> P1.13
- W4_16 pad 1: P1.15 -> P1.13
- W4_17 pad 1: P1.15 -> P1.13
- W4_18 pad 1: P1.15 -> P1.13
- W4_19 pad 1: P1.15 -> P1.13
- W4_20 pad 1: P1.15 -> P1.13
- W4_21 pad 1: P1.15 -> P1.13
- W4_22 pad 1: P1.15 -> P1.13
- W4_23 pad 1: P1.15 -> P1.13
- W4_24 pad 1: P1.15 -> P1.13
- W4_25 pad 1: P1.15 -> P1.13
- W4_26 pad 1: P1.15 -> P1.13
- W4_27 pad 1: P1.15 -> P1.13
- W4_28 pad 1: P1.15 -> P1.13
- W4_29 pad 1: P1.15 -> P1.13
- W4_30 pad 1: P1.15 -> P1.13
- W4_31 pad 1: P1.15 -> P1.13
- W4_32 pad 1: P1.15 -> P1.13
- W4_33 pad 1: P1.15 -> P1.13
- W4_34 pad 1: P1.15 -> P1.13
- W4_35 pad 1: P1.15 -> P1.13
- W5_01 pad 1: P0.03 -> P1.10
- W5_02 pad 1: P0.03 -> P1.10
- W5_03 pad 1: P0.03 -> P1.10
- W5_04 pad 1: P0.03 -> P1.10
- W5_05 pad 1: P0.03 -> P1.10
- W5_06 pad 1: P0.03 -> P1.10
- W5_07 pad 1: P0.03 -> P1.10
- W5_08 pad 1: P0.03 -> P1.10
- W5_09 pad 1: P0.03 -> P1.10
- W5_10 pad 1: P0.03 -> P1.10
- W5_11 pad 1: P0.03 -> P1.10
- W5_12 pad 1: P0.03 -> P1.10
- W5_13 pad 1: P0.03 -> P1.10
- W5_14 pad 1: P0.03 -> P1.10
- W5_15 pad 1: P0.03 -> P1.10
- W5_16 pad 1: P0.03 -> P1.10
- W5_17 pad 1: P0.03 -> P1.10
- W5_18 pad 1: P0.03 -> P1.10
- W5_19 pad 1: P0.03 -> P1.10
- W5_20 pad 1: P0.03 -> P1.10
- W5_21 pad 1: P0.03 -> P1.10
- W5_22 pad 1: P0.03 -> P1.10
- W5_23 pad 1: P0.03 -> P1.10
- W5_24 pad 1: P0.03 -> P1.10
- W5_25 pad 1: P0.03 -> P1.10
- W5_26 pad 1: P0.03 -> P1.10
- W5_27 pad 1: P0.03 -> P1.10
- W5_28 pad 1: P0.03 -> P1.10
- W5_29 pad 1: P0.03 -> P1.10
- W5_30 pad 1: P0.03 -> P1.10
- W5_31 pad 1: P0.03 -> P1.10
- W5_32 pad 1: P0.03 -> P1.10
- W5_33 pad 1: P0.03 -> P1.10
- W5_34 pad 1: P0.03 -> P1.10
- W5_35 pad 1: P0.03 -> P1.10
- W6_01 pad 1: P0.28 -> P0.03
- W6_02 pad 1: P0.28 -> P0.03
- W6_03 pad 1: P0.28 -> P0.03
- W6_04 pad 1: P0.28 -> P0.03
- W6_05 pad 1: P0.28 -> P0.03
- W6_06 pad 1: P0.28 -> P0.03
- W6_07 pad 1: P0.28 -> P0.03
- W6_08 pad 1: P0.28 -> P0.03
- W6_09 pad 1: P0.28 -> P0.03
- W6_10 pad 1: P0.28 -> P0.03
- W6_11 pad 1: P0.28 -> P0.03
- W6_12 pad 1: P0.28 -> P0.03
- W6_13 pad 1: P0.28 -> P0.03
- W6_14 pad 1: P0.28 -> P0.03
- W6_15 pad 1: P0.28 -> P0.03
- W6_16 pad 1: P0.28 -> P0.03
- W6_17 pad 1: P0.28 -> P0.03
- W6_18 pad 1: P0.28 -> P0.03
- W6_19 pad 1: P0.28 -> P0.03
- W6_20 pad 1: P0.28 -> P0.03
- W6_21 pad 1: P0.28 -> P0.03
- W6_22 pad 1: P0.28 -> P0.03
- W6_23 pad 1: P0.28 -> P0.03
- W6_24 pad 1: P0.28 -> P0.03
- W6_25 pad 1: P0.28 -> P0.03
- W6_26 pad 1: P0.28 -> P0.03
- W6_27 pad 1: P0.28 -> P0.03
- W6_28 pad 1: P0.28 -> P0.03
- W6_29 pad 1: P0.28 -> P0.03
- W6_30 pad 1: P0.28 -> P0.03
- W6_31 pad 1: P0.28 -> P0.03
- W6_32 pad 1: P0.28 -> P0.03
- W6_33 pad 1: P0.28 -> P0.03
- W6_34 pad 1: P0.28 -> P0.03
- W6_35 pad 1: P0.28 -> P0.03
- W7_01 pad 1: P0.12 -> P1.04
- W7_02 pad 1: P0.12 -> P1.04
- W7_03 pad 1: P0.12 -> P1.04
- W7_04 pad 1: P0.12 -> P1.04
- W7_05 pad 1: P0.12 -> P1.04
- W7_06 pad 1: P0.12 -> P1.04
- W7_07 pad 1: P0.12 -> P1.04
- W7_08 pad 1: P0.12 -> P1.04
- W7_09 pad 1: P0.12 -> P1.04
- W7_10 pad 1: P0.12 -> P1.04
- W7_11 pad 1: P0.12 -> P1.04
- W7_12 pad 1: P0.12 -> P1.04
- W7_13 pad 1: P0.12 -> P1.04
- W7_14 pad 1: P0.12 -> P1.04
- W7_15 pad 1: P0.12 -> P1.04
- W7_16 pad 1: P0.12 -> P1.04
- W7_17 pad 1: P0.12 -> P1.04
- W7_18 pad 1: P0.12 -> P1.04
- W7_19 pad 1: P0.12 -> P1.04
- W7_20 pad 1: P0.12 -> P1.04
- W7_21 pad 1: P0.12 -> P1.04
- W7_22 pad 1: P0.12 -> P1.04
- W7_23 pad 1: P0.12 -> P1.04
- W7_24 pad 1: P0.12 -> P1.04
- W7_25 pad 1: P0.12 -> P1.04
- W7_26 pad 1: P0.12 -> P1.04
- W7_27 pad 1: P0.12 -> P1.04
- W7_28 pad 1: P0.12 -> P1.04
- W7_29 pad 1: P0.12 -> P1.04
- W7_30 pad 1: P0.12 -> P1.04
- W7_31 pad 1: P0.12 -> P1.04
- W7_32 pad 1: P0.12 -> P1.04
- W7_33 pad 1: P0.12 -> P1.04
- W7_34 pad 1: P0.12 -> P1.04
- W7_35 pad 1: P0.12 -> P1.04
Routing:
- net USB_D+: track 937.1 -> 460.9 mm, vias 455 -> 350
- net P0.28: track 385.5 -> 0.00 mm, vias 35 -> 0
- net P1.13: track 0.00 -> 312.5 mm, vias 0 -> 70
- net DECUSB: track 358.8 -> 63.9 mm, vias 245 -> 35
- net P1.03: track 0.00 -> 244.9 mm, vias 0 -> 105
- net P1.04: track 244.9 -> 64.3 mm, vias 105 -> 70
- net P0.03: track 230.9 -> 385.5 mm, vias 70 -> 35
- net USB_D-: track 862.6 -> 758.2 mm, vias 315 -> 245
- net P0.12: track 64.3 -> 0.00 mm, vias 70 -> 0
- net P1.10: track 279.5 -> 230.9 mm
- net P1.15: track 312.5 -> 279.5 mm
- net P1.12: track 118.6 -> 135.5 mm, vias 0 -> 70
- net P1.11: track 135.5 -> 118.6 mm, vias 70 -> 0
- net GND: track 429.4 -> 441.3 mm, vias 1260 -> 1435
- net +3V3: track 388.3 -> 399.9 mm
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Other:
- board text added: "tabs NORTH EDGE ONLY, 2 x 5.000 mm per board, mouse bites 0.500 mm on 0.850 mm pitch, centres 0.500 mm into routed gap"
- board text removed: "C6 C3902158 10uF/10V; C19 C318563 4.7uF/16V; VDDH LOAD-STEP CHECK OPEN"
- board text removed: "CUSTOM WEST RADIATOR 0.850x7.435; EM/VNA REQUIRED"
- board text removed: "L4 RF FEED CORRIDOR; FIELD SOLVE REQUIRED"
- board text removed: "SIX-POSITION RF MATCH RESERVATION"
- board text removed: "tabs NORTH EDGE ONLY, 2 x 5.000 mm per board, mouse bites 0.600 mm on 0.850 mm pitch, centres 0.350 mm into routed gap"
