File: hw/meenie.kicad_pcb (KiCad board)
At the start: 8 copper layers, 13.6 x 9.4 mm, 50 parts, among them J1 USB-C 16P sink, SW1 GSNANOT000102, U1 nRF52840-QIAA-R, Y1 FA-118T 32MHz CL 8pF

Commit message: Fab Ready
Parts:
- C21: value 820pF -> 820pF C0G 5%
- C6: value 10uF -> 4.7uF; footprint meenie:C0402 -> meenie:C0603
- C8: value 1.0uF -> 100nF
- D1, D4: moved to F.Cu
- D2: value TPD1E6B06DPLR -> ESD441DPLR
- moved D4 7.46 mm to (107.5, 92.5), turned to -90 degrees
- moved D1 7.19 mm to (108.1, 92.5), turned to 90 degrees
- moved D2 5.64 mm to (109.7, 92.5)
- moved C6 0.28 mm to (101.7, 95.6)
- moved D3 0.07 mm to (113.0, 96.3)
Connections:
- net P0.05 renamed P1.05
- net P0.11 renamed P1.06
- net P0.13 renamed P1.01
- net P0.27 renamed P1.07
- net P0.31 renamed P0.02
- E6 pad 1: P1.04 -> P1.03
- E8 pad 1: P1.10 -> P1.15
- E9 pad 1: P1.11 -> P1.12
- U1 pad A14: P1.10 -> P1.15
- U1 pad A16: P1.15 -> P1.13
- U1 pad A20: P0.03 -> P1.10
- U1 pad B13: P0.28 -> P0.03
- U1 pad B17: P1.11 -> P1.12
- U1 pad B19: P1.12 -> P1.11
- U1 pad U24: P0.12 -> P1.04
- U1 pad V23: P1.04 -> P1.03
- W2 pad 1: P1.12 -> P1.11
- W4 pad 1: P1.15 -> P1.13
- W5 pad 1: P0.03 -> P1.10
- W6 pad 1: P0.28 -> P0.03
- W7 pad 1: P0.12 -> P1.04
Routing:
- net USB_D+: track 26.8 -> 13.2 mm, vias 13 -> 10
- net P0.28: track 11.0 -> 0.00 mm, vias 1 -> 0
- net P1.13: track 0.00 -> 8.93 mm, vias 0 -> 2
- net DECUSB: track 10.3 -> 1.83 mm, vias 7 -> 1
- net P1.03: track 0.00 -> 7.00 mm, vias 0 -> 3
- net P1.04: track 7.00 -> 1.84 mm, vias 3 -> 2
- net P0.03: track 6.60 -> 11.0 mm, vias 2 -> 1
- net USB_D-: track 24.6 -> 21.7 mm, vias 9 -> 7
- net P0.12: track 1.84 -> 0.00 mm, vias 2 -> 0
- net P1.10: track 7.99 -> 6.60 mm
- net P1.15: track 8.93 -> 7.99 mm
- net P1.12: track 3.39 -> 3.87 mm, vias 0 -> 2
- net P1.11: track 3.87 -> 3.39 mm, vias 2 -> 0
- net GND: track 12.3 -> 12.6 mm, vias 36 -> 41
Other:
- board text removed: "C6 C3902158 10uF/10V; C19 C318563 4.7uF/16V; VDDH LOAD-STEP CHECK OPEN"
- board text removed: "CUSTOM WEST RADIATOR 0.850x7.435; EM/VNA REQUIRED"
- board text removed: "L4 RF FEED CORRIDOR; FIELD SOLVE REQUIRED"
- board text removed: "SIX-POSITION RF MATCH RESERVATION"
