File: hw/meenie.kicad_sch (KiCad schematic)
At the start: 51 parts, among them J1 USB-C 16P sink, SW1 GSNANOT000102, U1 nRF52840-QIAA-R, Y1 FA-118T 32MHz CL 8pF

Commit message: Fab Ready
Parts:
- C11, C9: LCSC Part C69335 -> C90057; MPN (none) -> GRM188R61E475KE11D; Manufacturer (none) -> Murata Electronics
- C12, C18, C3: MPN (none) -> GRM033C71C104KE14D; Manufacturer (none) -> Murata Electronics
- C14, C16: MPN (none) -> GJM0335C1ER80WB01D; Manufacturer (none) -> Murata Electronics
- C15: MPN (none) -> GJM0335C1HR50WB01D; Manufacturer (none) -> Murata Electronics
- C19: MPN (none) -> CL05A475MO5NUNC; Manufacturer (none) -> Samsung Electro-Mechanics
- C21: value 820pF -> 820pF C0G 5%; LCSC Part C185597 -> C384953; MPN (none) -> GRM0335C1E821JA01D; Manufacturer (none) -> Murata Electronics
- C5: MPN (none) -> CC0201JRNPO9BN101; Manufacturer (none) -> Yageo
- C6: value 10uF -> 4.7uF; footprint meenie:C0402 -> meenie:C0603; LCSC Part C3902158 -> C90057; MPN (none) -> GRM188R61E475KE11D; Manufacturer (none) -> Murata Electronics; Manufacturer Part Number CL05A106MP6NUN8 -> GRM188R61E475KE11D
- C7: MPN (none) -> CL05A105KA5NQNC; Manufacturer (none) -> Samsung Electro-Mechanics
- C8: value 1.0uF -> 100nF; LCSC Part C52923 -> C1525; MPN (none) -> CL05B104KO5NNNC; Manufacturer (none) -> Samsung Electro-Mechanics; Manufacturer Part Number (none) -> CL05B104KO5NNNC
- D2: value TPD1E6B06DPLR -> ESD441DPLR; LCSC Part C914099 -> C22427765; MPN TPD1E6B06DPLR -> ESD441DPLR
- D3: MPN (none) -> LTST-C281KRKT; Manufacturer (none) -> Lite-On
- L1, L2: MPN (none) -> LQP03HQ4N7H02D; Manufacturer (none) -> Murata Electronics
- R1: MPN (none) -> RC0402FR-072R2L; Manufacturer (none) -> Yageo
- R2, R3: LCSC Part C270344 -> C274341; MPN (none) -> RC0201FR-075K1L; Manufacturer (none) -> Yageo
- R4: MPN (none) -> 0201WMF1001TEE; Manufacturer (none) -> Uniroyal Electronics
Connections:
- net P0.12 is gone; now on net P1.04: U1.U24 (P1.04), W7.1
- net P0.28 is gone; now on net P0.03: U1.B13 (P0.03/AIN1), W6.1
- net P0.03: no longer U1.A20 (P1.10), W5.1
- net P1.04: no longer E6.1, U1.V23 (P1.03)
- net P1.10: now also U1.A20 (P1.10), W5.1; no longer E8.1, U1.A14 (P1.15)
- net P1.11: now also U1.B19 (P1.11), W2.1; no longer E9.1, U1.B17 (P1.12)
- net P1.12: now also E9.1, U1.B17 (P1.12); no longer U1.B19 (P1.11), W2.1
- net P1.15: now also E8.1, U1.A14 (P1.15); no longer U1.A16 (P1.13), W4.1
- net P0.05 renamed P1.05
- net P0.11 renamed P1.06
- net P0.13 renamed P1.01
- net P0.27 renamed P1.07
- net P0.31 renamed P0.02
- new net P1.03: E6.1, U1.V23 (P1.03)
- new net P1.13: U1.A16 (P1.13), W4.1
Other:
- note removed: "3.3 V output. Never drive the 3V3 pad from outside."
- note removed: "3.3 V, so green and blue are out at 2.5 to 3.6 V of Vf. Red or yellow-green only."
- note removed: "32 MHz HFXO. Y1 is 32.000 MHz, CL 8 pF, FA-118T 1612 four pad."
- note removed: "AIN7 E3. AIN2 on J1 is the one channel no breakout pad carries."
- note removed: "ANT_FEED ends at AE1, a custom 0.850 x 7.435 mm F.Cu radiator requiring EM and VNA validation."
- note removed: "APPROTECT follows the build code shipped under the -R order code. Dxx and earlier"
- note removed: "C1 and C2 are the 12 pF NP0 2% load capacitors. No LFXO: the calibrated LFRC"
- note removed: "C14 returns to U1 pin F23 VSS_PA and not to the plane. F23 is a ground pin and sits"
- note removed: "C18 X7R 10% 0201, C5 NP0 5% 0201, C7 X7R 10% 0402, C21 NP0 5% 0201, C9 X7S 10% 0603."
- note removed: "C21 is fitted on build codes Dxx and earlier, which is what the -R order code ships."
- note removed: "C3, C4 and C12 are X7R 10% 0201, C8 is X7R 10% 0402, C6 is X7R 10% 0603."
- note removed: "Capacitors C0G 0201, inductors HF chip 0201. C16 is fitted; C17 is the DNP feed-side tuning position."
- note removed: "D1 and D4 are the dedicated low-capacitance USB ESD protectors. No series resistors: the USB"
- note removed: "D1 pin 1 is D+, D4 pin 2 is D-, and each remaining pin is the shortest available ground."
- note removed: "DEC2 carries no external part in that configuration. DEC4 must be tied to DEC6."
- note removed: "ESD5311Z-2/TR is fitted once per data net in its vendor DFN0603-2 land pattern."
- note removed: "GND and VBUS_MCU have no driving pin anywhere on the sheet, so each one carries a flag."
- note removed: "High voltage mode is a wiring decision and not a register write. VBUS reaches VDDH"
- note removed: "Internal regulator decoupling, Nordic circuit configuration 1 for the aQFN73."
- note removed: "It is not required on Fxx and later. C9 carries CDECUSB, 2.35 uF minimum after bias."
- note removed: "Never enable the DC/DC regulator. There is no external LC filter on this board and"
- note removed: "PSELRESET. The E7 pad is P0.18 and is a plain GPIO until UICR.PSELRESET[0] at 0x200"
- note removed: "R2 and R3 are 5.1k 1%. R1 is 2R2 1% 0.063W and eats 2.2 of the 3.8 ohm source"
- note removed: "REGOUT0. UICR.REGOUT0.VOUT must be written to 3.3 V, field value 5 at offset 0x304."
- note removed: "SAADC capable, two grounds, 3V3 out, VBUS in and unfused, nRESET for double-tap DFU,"
- note removed: "SoC match then antenna pi. Order out of the ANT pin: C14 shunt, L1 series, C15 shunt,"
- note removed: "Status LED on P1.02, R4 1k in series, cathode pin 1 to GND. Red, Vf 2.0 V. The rail is"
- note removed: "The factory default is 1.8 V, so a board that skips the write brings every GPIO and"
- note removed: "The match is Nordic configuration 1 for the aQFN73, three components: C14 0.8 pF"
- note removed: "Twenty surface pads on B.Cu, 0.60 mm square. W1 to W9 with S1 and S2 sit on the north"
- note removed: "UICR, so the write has to be repeated after any debug recovery."
- note removed: "USB-C receptacle wired as a sink. Two Rd, one per CC, because a plug can seat"
- note removed: "VDD decoupling. REG0 sources this rail in high voltage mode, so VDD is an output here."
- note removed: "access until a filter is fitted. DCC and DCCH stay open and no inductor is fitted."
- note removed: "and PSELRESET[1] at 0x204 both read 18. Until then the pad does nothing and the only"
- note removed: "and the two SWD pads. Every GPIO sits on a U1 pin with a measured via-in-pad seat, so"
- note removed: "attach over SWD with no ERASEALL; Fxx and later need an ERASEALL through CTRL-AP"
- note removed: "configuration 7, the battery DC/DC arrangement, and they are struck. Nordic draws a"
- note removed: "either way up. D+ reaches A6 and B6, D- reaches A7 and B7, for the same reason."
- note removed: "first, then UICR.APPROTECT plus the APPROTECT.DISABLE register on every boot."
- note removed: "holds 500 ppm, which is exactly the BLE sleep clock requirement."
- note removed: "on GND, as Nordic draws it. The routing is what filters harmonics, not a split net."
- note removed: "peripheral makes its own 3.3 V from VBUS for signalling and for the D+ pull-up."
- note removed: "rail at y 9.000, E1 to E9 on the east rail at x 12.100. Thirteen GPIO, seven of them"
- note removed: "resistance budget. C11 is X7R 10% and C19 X7S 10%, both 0603. D2 is a 6 V"
- note removed: "shunt, L1 4.7 nH series, C15 0.5 pF shunt, NP0 at plus or minus 10 percent. That is"
- note removed: "the 3V3 pad up at 1.8 V and browns out under load. ERASEALL and --recover both wipe"
- note removed: "the configuration whose supply topology this board has, VDDH from VBUS on the LDO"
- note removed: "the escape is a drop onto In2. AIN0 E5, AIN1 W5, AIN3 E2, AIN4 W6, AIN5 E4, AIN6 W7,"
- note removed: "then the pi C16 shunt and L2 series into the etched radiator."
- note removed: "there is not going to be one; enabling it inhibits device operation including debug"
- note removed: "third shunt C22 on the same node and leaves it unmounted; C16 already sits there."
- note removed: "through R1 and nothing drives VDD, so REG0 regulates VDDH down and VDD becomes the"
- note removed: "unidirectional clamp on the bare VBUS pad."
- note removed: "way in is SWD. ERASEALL wipes it alongside REGOUT0, so both get rewritten together."
- note removed: "with no DC/DC and no NFC. The four component values that stood here are Nordic"
